Commit message: Changing find package command to point to Final-year-project in sjtu_drone.urdf as it causes error when running simple.launch

File: urdf/sjtu_drone.urdf (robot description, URDF)
Before this commit: robot sjtu_drone, 1 links, 0 joints
Links:
- link base_link: geometry collision mesh filename=package://Final-year-project/meshes/quadrotor_4.stl; visual mesh filename=package://Final-year-project/meshes/quadrotor_4.dae

Commit message: Manual merge of NOVOG93 and my own repos to have an updated system

File: urdf/sjtu_drone.urdf (robot description, URDF)
Before this commit: robot sjtu_drone, 1 links, 0 joints
Links:
- link base_link: geometry collision mesh filename=package://sjtu_drone/meshes/quadrotor_4.stl; visual mesh filename=package://sjtu_drone/meshes/quadrotor_4.dae
